File: kicad-pmod_i2s2.kicad_sch (KiCad schematic)
At the start: 0 parts

Commit message: made schematic and draft placement
Parts:
- added C? (x7): 100n, Capacitor_SMD:C_0603_1608Metric_Pad1.08x0.95mm_HandSolder, symbol Device:C
- added C? (x3): 10u, Capacitor_SMD:C_0603_1608Metric_Pad1.08x0.95mm_HandSolder, symbol Device:C
- added C? (x3): 1u, Capacitor_SMD:C_0603_1608Metric_Pad1.08x0.95mm_HandSolder, symbol Device:C
- added C? (x2): 2n7, Capacitor_SMD:C_0603_1608Metric_Pad1.08x0.95mm_HandSolder, symbol Device:C
- added C? (x2): 4u7, Capacitor_SMD:C_0603_1608Metric_Pad1.08x0.95mm_HandSolder, symbol Device:C
- added C? (x2): 3u3, Capacitor_SMD:C_0603_1608Metric_Pad1.08x0.95mm_HandSolder, symbol Device:C
- added C? (x2): 180p, Capacitor_SMD:C_0603_1608Metric_Pad1.08x0.95mm_HandSolder, symbol Device:C
- added FB1, FB2: 600, Inductor_SMD:L_0603_1608Metric_Pad1.05x0.95mm_HandSolder, symbol Device:FerriteBead
- added J1: M/S, Connector_PinHeader_2.54mm:PinHeader_1x03_P2.54mm_Vertical, symbol Connector:Conn_01x03_Pin
- added J?: Audio In, Connector_Audio:Jack_3.5mm_PJ320D_Horizontal, symbol Connector:AudioJack4
- added J?: Audio Out, Connector_Audio:Jack_3.5mm_PJ320D_Horizontal, symbol Connector:AudioJack4
- added J?: pmod, Connector_PinHeader_2.54mm:PinHeader_2x06_P2.54mm_Horizontal, symbol Connector_Generic:Conn_02x06_Odd_Even
- added R? (x2): 470, Resistor_SMD:R_0603_1608Metric_Pad0.98x0.95mm_HandSolder, symbol Device:R
- added R? (x4): 5k1, Resistor_SMD:R_0603_1608Metric_Pad0.98x0.95mm_HandSolder, symbol Device:R
- added R? (x3): 10k, Resistor_SMD:R_0603_1608Metric_Pad0.98x0.95mm_HandSolder, symbol Device:R
- added R?: 0, Resistor_SMD:R_0603_1608Metric_Pad0.98x0.95mm_HandSolder, symbol Device:R
- added U1: 74LVC1G126, Package_TO_SOT_SMD:SOT-23-5_HandSoldering, symbol 74xGxx:74AHC1G126
- added U2: CS4344, Package_SO:TSSOP-10_3x3mm_P0.5mm, symbol Audio:CS4344
- added U3: CS5343, Package_SO:TSSOP-10_3x3mm_P0.5mm, symbol Audio:CS5343
Connections:
- new net: C?.1, C?.1, U2.5 (VQ)
- new net: C?.1, U2.10 (AOUTR)
- new net: C?.1, U2.6 (FILT+)
- new net: C?.1, U2.7 (AOUTL)
- new net: C?.1, C?.1, FB1.2, U2.9 (VA)
- new net: C?.2, R?.1, R?.1 (x4)
- new net: C?.1, J?.T, R?.2
- new net: C?.1, U3.5 (FILT+)
- new net: J?.R1, R?.2
- new net: J?.T, R?.2
- new net: C?.1, C?.1, FB2.2, U3.10 (VA)
- new net: C?.1, C?.1, U3.8 (AINR)
- new net: C?.1, J?.R1, R?.2
- new net: C?.1, C?.1, U3.6 (AINL)
- new net: C?.1, C?.1, U3.7 (VQ)
- new net: J1.2 (Pin_2), R?.2
- new net: R?.1, U1.4
- new net +3V3: C?.1, C?.1, C?.1, FB1.1, FB2.1, J1.1 (Pin_1), J?.11 (Pin_11), J?.12 (Pin_12), U1.1, U1.5 (VCC)
- new net ADIN_LRCLK: J?.4 (Pin_4), U3.3 (LRCK)
- new net ADIN_MCLK: J?.2 (Pin_2), U3.4 (MCLK)
- new net ADIN_SCLK: J?.6 (Pin_6), U3.2 (SCLK)
- new net ADIN_SDOUT: J?.8 (Pin_8), R?.2
- new net ADOUT_LRCLK: J?.3 (Pin_3), U2.3 (LRCK)
- new net ADOUT_MCLK: J?.1 (Pin_1), U2.4 (MCLK)
- new net ADOUT_SCLK: J?.5 (Pin_5), U2.2 (~{DEM}/SCLK)
- new net ADOUT_SDIN: J?.7 (Pin_7), U2.1 (SDIN)
- new net GND: C?.2, C?.2, C?.2, C?.2, C?.2, C?.2, C?.2, C?.2, C?.2, C?.2, C?.2, C?.2, C?.2, C?.2, C?.2, C?.2, C?.2, J1.3 (Pin_3), J?.10 (Pin_10), J?.9 (Pin_9), J?.S, J?.S, R?.2, R?.2, R?.2, R?.2, U1.3 (GND), U2.8 (GND), U3.9 (GND)
- new net SDOUT: R?.1, U1.2, U3.1 (SDOUT)
- no-connect marks 0 -> 2
Other:
- note added: "Jumper Settings Master: 1-2 Slave: 3-2"

Commit message: update ADC capacitors properties
Parts:
- removed C?: 180p, Capacitor_SMD:C_0603_1608Metric_Pad1.08x0.95mm_HandSolder, symbol Device:C
- added C?: 180p, Capacitor_SMD:C_0603_1608Metric_Pad1.08x0.95mm_HandSolder, symbol Device:C
- C?: Type (none) -> NPO
Connections:
- net GND: now also C?.2
- net at C?.1, U3.6 (AINL): now also C?.1
Changed lines of the file:
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@@
+    )
+  )
+  (symbol (lib_id "Device:C") (at 194.31 137.16 0) (unit 1)
+    (in_bom yes) (on_board yes) (dnp no)
+    (property "Reference" "C?" (at 198.12 135.89 0)
+      (effects (font (size 1.27 1.27)) (justify left))
+    )
+    (property "Value" "180p" (at 198.12 138.43 0)
+      (effects (font (size 1.27 1.27)) (justify left))
+    )
+    (property "Footprint" "Capacitor_SMD:C_0603_1608Metric_Pad1.08x0.95mm_HandSolder" (at 195.2752 140.97 0)
+      (effects (font (size 1.27 1.27)) hide)
+    )
+    (property "Datasheet" "~" (at 194.31 137.16 0)
+      (effects (font (size 1.27 1.27)) hide)
+    )
+    (property "Type" "NPO" (at 198.12 140.97 0)
+      (effects (font (size 1.27 1.27)) (justify left))
+    )
+    (pin "1")
+    (pin "2")
+    (instances
+      (project "pcm_pmod"
+        (path "/5b4b9bd4-3915-4731-81a6-668a66ef2261"
+          (reference "C?") (unit 1)
+        )
+      )
+      (project "kicad-pmod_i2s2"
+        (path "/cca618d6-30d1-42b0-bf93-86ddd5d8c9e4"
+          (reference "C17") (unit 1)
+        )
+      )
     )
   )
@@
   )
   (symbol (lib_id "Device:C") (at 181.61 137.16 0) (unit 1)
-    (in_bom yes) (on_board yes) (dnp no) (fields_autoplaced)
+    (in_bom yes) (on_board yes) (dnp no)
     (property "Reference" "C?" (at 185.42 135.89 0)
       (effects (font (size 1.27 1.27)) (justify left))
@@
       (effects (font (size 1.27 1.27)) hide)
     )
+    (property "Type" "NPO" (at 185.42 140.97 0)
+      (effects (font (size 1.27 1.27)) (justify left))
+    )
     (pin "1")
     (pin "2")
@@
         )
       )
-    )
-  )
-  (symbol (lib_id "Device:C") (at 194.31 137.16 0) (unit 1)
-    (in_bom yes) (on_board yes) (dnp no) (fields_autoplaced)
-    (property "Reference" "C?" (at 198.12 135.89 0)
-      (effects (font (size 1.27 1.27)) (justify left))
-    )
-    (property "Value" "180p" (at 198.12 138.43 0)
-      (effects (font (size 1.27 1.27)) (justify left))
-    )
-    (property "Footprint" "Capacitor_SMD:C_0603_1608Metric_Pad1.08x0.95mm_HandSolder" (at 195.2752 140.97 0)
-      (effects (font (size 1.27 1.27)) hide)
-    )
-    (property "Datasheet" "~" (at 194.31 137.16 0)
-      (effects (font (size 1.27 1.27)) hide)
-    )
-    (pin "1")
-    (pin "2")
-    (instances
-      (project "pcm_pmod"
-        (path "/5b4b9bd4-3915-4731-81a6-668a66ef2261"
-          (reference "C?") (unit 1)
-        )
-      )
-      (project "kicad-pmod_i2s2"
-        (path "/cca618d6-30d1-42b0-bf93-86ddd5d8c9e4"
-          (reference "C17") (unit 1)
-        )
-      )
